File: indicator/pcb/helioHydration_indicator.kicad_pcb (KiCad board)
At the start: 2 copper layers, 50 x 50 mm, 16 parts, among them U1 DS18B20, U2 GUVA-S12SD, U3 ATmega328P-P, U4 LM7805_TO220, U5 4-Wire-SPI, Y1 CrystalOscillator_16MHz

Commit message: make indicator housing
Parts:
- moved U4 7.89 mm to (170.4, 75.3), turned to 180 degrees
- moved C3 7.68 mm to (177.5, 85.6), turned to 90 degrees
- moved C4 7.54 mm to (177.5, 92.0), turned to 90 degrees
Routing:
- net GND_REG: track 80.3 -> 98.5 mm
- net 5V_REG: track 111.5 -> 119.9 mm
- net 8-12V: track 7.39 -> 14.7 mm

Commit message: update pcb
Parts:
- added REF**: power_input, Arduino_ISPProgrammer:power_input, F.Cu at (177.1, 102.3)
Routing:
- net GND_REG: track 98.5 -> 121.2 mm
- net 8-12V: track 14.7 -> 31.9 mm, vias 0 -> 1
Changed lines of the file:
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@@
 			(drillshape 0)
 			(scaleselection 1)
-			(outputdirectory "production/")
+			(outputdirectory "production/gerbers/")
 		)
 	)
@@
 		)
 	)
+	(footprint "Arduino_ISPProgrammer:power_input"
+		(layer "F.Cu")
+		(at 177.134 102.317)
+		(property "Reference" "REF**"
+			(at 0 -0.5 0)
+			(unlocked yes)
+			(layer "F.SilkS")
+			(effects
+				(font
+					(size 1 1)
+					(thickness 0.1)
+				)
+			)
+		)
+		(property "Value" "power_input"
+			(at 0 1 0)
+			(unlocked yes)
+			(layer "F.Fab")
+			(effects
+				(font
+					(size 1 1)
+					(thickness 0.15)
+				)
+			)
+		)
+		(property "Datasheet" ""
+			(at 0 0 0)
+			(unlocked yes)
+			(layer "F.Fab")
+			(hide yes)
+			(effects
+				(font
+					(size 1 1)
+					(thickness 0.15)
+				)
+			)
+		)
+		(property "Description" ""
+			(at 0 0 0)
+			(unlocked yes)
+			(layer "F.Fab")
+			(hide yes)
+			(effects
+				(font
+					(size 1 1)
+					(thickness 0.15)
+				)
+			)
+		)
+		(attr smd)
+		(fp_rect
+			(start -1.85 -3.2)
+			(end 1.85 3.2)
+			(stroke
+				(width 0.1)
+				(type default)
+			)
+			(fill no)
+			(layer "F.SilkS")
+		)
+		(fp_text user "${REFERENCE}"
+			(at 0 2.5 0)
+			(unlocked yes)
+			(layer "F.Fab")
+			(effects
+				(font
+					(size 1 1)
+					(thickness 0.15)
+				)
+			)
+		)
+		(pad "1" thru_hole circle
+			(at 0 -1.24)
+			(size 1.6 1.6)
+			(drill 1)
+			(layers "*.Cu" "*.Mask")
+			(remove_unused_layers no)
+			(net 4 "8-12V")
+		)
+		(pad "2" thru_hole circle
+			(at 0 1.3)
+			(size 1.6 1.6)
+			(drill 1)
+			(layers "*.Cu" "*.Mask")
+			(remove_unused_layers no)
+			(net 2 "GND_REG")
+		)
+		(embedded_fonts no)
+	)
 	(footprint "Capacitor_SMD:C_1206_3216Metric"
 		(layer "F.Cu")
@@
 	)
 	(segment
+		(start 179.587 84.112)
+		(end 177.466 84.112)
+		(width 0.2)
+		(layer "F.Cu")
+		(net 2)
+	)
+	(segment
+		(start 179.637 101.114)
+		(end 179.637 84.162)
+		(width 0.2)
+		(layer "F.Cu")
+		(net 2)
+	)
+	(segment
 		(start 168.621 98.431)
 		(end 168.01 97.82)
@@
 	)
 	(segment
+		(start 179.637 84.162)
+		(end 179.587 84.112)
+		(width 0.2)
+		(layer "F.Cu")
+		(net 2)
+	)
+	(segment
 		(start 171.544 98.431)
 		(end 168.621 98.431)
@@
 	)
 	(segment
+		(start 177.134 103.617)
+		(end 179.637 101.114)
+		(width 0.2)
+		(layer "F.Cu")
+		(net 2)
+	)
+	(segment
 		(start 155.760079 86.174921)
 		(end 155.760079 79.094579)
@@
 	)
 	(segment
+		(start 175.536 87.062)
+		(end 177.466 87.062)
+		(width 0.2)
+		(layer "F.Cu")
+		(net 4)
+	)
+	(segment
+		(start 174.998 87.6)
+		(end 175.536 87.062)
+		(width 0.2)
+		(layer "F.Cu")
+		(net 4)
+	)
+	(segment
 		(start 170.449 75.255)
 		(end 170.449 80.045)
@@
 		(net 4)
 	)
+	(via
+		(at 174.998 87.6)
+		(size 0.6)
+		(drill 0.3)
+		(layers "F.Cu" "B.Cu")
+		(net 4)
+	)
+	(segment
+		(start 177.134 89.537)
+		(end 177.134 101.077)
+		(width 0.2)
+		(layer "B.Cu")
+		(net 4)
+	)
+	(segment
+		(start 174.998 87.6)
+		(end 175.197 87.6)
+		(width 0.2)
+		(layer "B.Cu")
+		(net 4)
+	)
+	(segment
+		(start 175.197 87.6)
+		(end 177.134 89.537)
+		(width 0.2)
+		(layer "B.Cu")
+		(net 4)
+	)
